File: pcb/65C816-CHIPz-module/65C816-CHIPz-module.kicad_pcb (KiCad board)
At the start: 2 copper layers, 63 x 22.5 mm, 29 parts, among them U1 W65C816, U2 74AHC1G00

Commit message: Add note to board.
Other:
- board text added: "Update QFP with CM_packages part for rev.B"
Changed lines of the file:
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@@
+		)
+	)
+	(gr_text "Update QFP with CM_packages part for rev.B"
+		(at 143 87 0)
+		(layer "Dwgs.User")
+		(effects
+			(font
+				(size 1 1)
+				(thickness 0.1)
+			)
+			(justify left bottom)
 		)
 	)
